Commit message: robot is almost able to stand - no tsid wrapper

File: ainex_project/install/ainex_description/share/ainex_description/robots/ainex.urdf.xacro (robot description, xacro)
@@ -1,1453 +1 @@
-<?xml version="1.0" encoding="utf-8"?>
-<robot name="ainex" xmlns:xacro="http://ros.org/wiki/xacro">
-  <xacro:property name="M_PI" value="3.1415926535897931" />
-  <xacro:include filename="$(find ainex_description)/urdf/materials.xacro" />
-  <xacro:include filename="$(find ainex_description)/urdf/transmissions.xacro" />
-  <xacro:property name="motor_torque" value="6"/>
-  <xacro:property name="motor_vec" value="100"/>
-  <xacro:property name="damping" value="0.02"/>
-  <xacro:property name="friction" value="0.0"/>
-  <xacro:property name="arm_damping" value="0.0"/>
-  <xacro:property name="arm_friction" value="0.2"/>
-  <link name="base_link"/>
-  <joint name="base_link_to_body" type="fixed">
-    <parent link="base_link"/>
-    <child link="body_link"/>
-  </joint>
-  <link
-    name="body_link">
-    <inertial>
-      <origin
-        xyz="0.00394313682998006 -7.92910841109997E-05 0.0504544952747596"
-        rpy="0 0 0" />
-      <mass
-        value="0.743" />
-      <inertia
-        ixx="0.00121619"
-        ixy="0.00000248"
-        ixz="-0.00005348"
-        iyy="0.00104402"
-        iyz="-0.00000200"
-        izz="0.00108564" />
-    </inertial>
-    <visual>
-      <origin
-        xyz="0 0 0"
-        rpy="0 0 0" />
-      <geometry>
-        <mesh
-          filename="package://ainex_description/meshes/body_link.STL" />
-      </geometry>
-      <material name="black"/>
-    </visual>
-    <collision>
-      <origin
-        xyz="0 0 0"
-        rpy="0 0 0" />
-      <geometry>
-        <mesh
-          filename="package://ainex_description/meshes/body_link.STL" />
-      </geometry>
-    </collision>
-  </link>
-  <link
-    name="r_hip_yaw_link">
-    <inertial>
-      <origin
-        xyz="-3.08089321559763E-05 0.0012572746209485 -0.00137106654438882"
-        rpy="0 0 0" />
-      <mass
-        value="0.032" />
-      <inertia
-        ixx="0.00001756"
-        ixy="-0.00000028"
-        ixz="-0.00000033"
-        iyy="0.00002270"
-        iyz="0.00000092"
-        izz="0.00000905" />
-    </inertial>
-    <visual>
-      <origin
-        xyz="0 0 0"
-        rpy="0 0 0" />
-      <geometry>
-        <mesh
-          filename="package://ainex_description/meshes/r_hip_yaw_link.STL" />
-      </geometry>
-      <material name="black"/>
-    </visual>
-    <collision>
-      <origin
-        xyz="0 0 0"
-        rpy="0 0 0" />
-      <geometry>
-        <mesh
-          filename="package://ainex_description/meshes/r_hip_yaw_link.STL" />
-      </geometry>
-    </collision>
-  </link>
-  <joint
-    name="r_hip_yaw"
-    type="revolute">
-    <origin
-      xyz="0 -0.029 0"
-      rpy="0 0 0" />
-    <parent
-      link="body_link" />
-    <child
-      link="r_hip_yaw_link" />
-    <axis
-      xyz="0 0 -1" />
-    <limit
-      lower="-2.09"
-      upper="2.09"
-      effort="${motor_torque}"
-      velocity="${motor_vec}" />
-    <dynamics
-      damping="${damping}"
-      friction="${friction}" />
-  </joint>
-  <link
-    name="r_hip_roll_link">
-    <inertial>
-      <origin
-        xyz="0.00136240189123019 -0.000566876191787073 -0.0134186815024998"
-        rpy="0 0 0" />
-      <mass
-        value="0.120" />
-      <inertia
-        ixx="0.00002918"
-        ixy="-0.00000090"
-        ixz="-0.00000045"
-        iyy="0.00007310"
-        iyz="0.00000000"
-        izz="0.00006050" />
-    </inertial>
-    <visual>
-      <origin
-        xyz="0 0 0"
-        rpy="0 0 0" />
-      <geometry>
-        <mesh
-          filename="package://ainex_description/meshes/r_hip_roll_link.STL" />
-      </geometry>
-      <material name="black"/>
-    </visual>
-    <collision>
-      <origin
-        xyz="0 0 0"
-        rpy="0 0 0" />
-      <geometry>
-        <mesh
-          filename="package://ainex_description/meshes/r_hip_roll_link.STL" />
-      </geometry>
-    </collision>
-  </link>
-  <joint
-    name="r_hip_roll"
-    type="revolute">
-    <origin
-      xyz="-0.01955 0 -0.0255"
-      rpy="0 0 0" />
-    <parent
-      link="r_hip_yaw_link" />
-    <child
-      link="r_hip_roll_link" />
-    <axis
-      xyz="-1 0 0" />
-    <limit
-      lower="-2.09"
-      upper="2.09"
-      effort="${motor_torque}"
-      velocity="${motor_vec}" />
-    <dynamics
-      damping="${damping}"
-      friction="${friction}" />
-  </joint>
-  <link
-    name="r_hip_pitch_link">
-    <inertial>
-      <origin
-        xyz="0.0135944229510165 0.0193812364621979 -0.0727053786154678"
-        rpy="0 0 0" />
-      <mass
-        value="0.1065" />
-      <inertia
-        ixx="0.00011009"
-        ixy="0.00000025"
-        ixz="-0.00000822"
-        iyy="0.00011292"
-        iyz="0.00000058"
-        izz="0.00004163" />
-    </inertial>
-    <visual>
-      <origin
-        xyz="0 0 0"
-        rpy="0 0 0" />
-      <geometry>
-        <mesh
-          filename="package://ainex_description/meshes/r_hip_pitch_link.STL" />
-      </geometry>
-      <material name="black"/>
-    </visual>
-    <collision>
-      <origin
-        xyz="0 0 0"
-        rpy="0 0 0" />
-      <geometry>
-        <mesh
-          filename="package://ainex_description/meshes/r_hip_pitch_link.STL" />
-      </geometry>
-    </collision>
-  </link>
-  <joint
-    name="r_hip_pitch"
-    type="revolute">
-    <origin
-      xyz="0.0190366011774447 -0.0200000000007891 0"
-      rpy="0 0 0" />
-    <parent
-      link="r_hip_roll_link" />
-    <child
-      link="r_hip_pitch_link" />
-    <axis
-      xyz="0 -1 0" />
-    <limit
-      lower="-2.09"
-      upper="2.09"
-      effort="${motor_torque}"
-      velocity="${motor_vec}" />
-    <dynamics
-      damping="${damping}"
-      friction="${friction}" />
-  </joint>
-  <link
-    name="r_knee_link">
-    <inertial>
-      <origin
-        xyz="0.00334266052421815 0.0196473707822286 -0.0425048961212657"
-        rpy="0 0 0" />
-      <mass
-        value="0.045" />
-      <inertia
-        ixx="0.00006733"
-        ixy="0.00000005"
-        ixz="0.00000285"
-        iyy="0.00005500"
-        iyz="0.00000000"
-        izz="0.00002073" />
-    </inertial>
-    <visual>
-      <origin
-        xyz="0 0 0"
-        rpy="0 0 0" />
-      <geometry>
-        <mesh
-          filename="package://ainex_description/meshes/r_knee_link.STL" />
-      </geometry>
-      <material name="black"/>
-    </visual>
-    <collision>
-      <origin
-        xyz="0 0 0"
-        rpy="0 0 0" />
-      <geometry>
-        <mesh
-          filename="package://ainex_description/meshes/r_knee_link.STL" />
-      </geometry>
-    </collision>
-  </link>
-  <joint
-    name="r_knee"
-    type="revolute">
-    <origin
-      xyz="-0.000372039419212393 4.99999999942422E-05 -0.0968862318156413"
-      rpy="0 0 0" />
-    <parent
-      link="r_hip_pitch_link" />
-    <child
-      link="r_knee_link" />
-    <axis
-      xyz="0 -1 0" />
-    <limit
-      lower="-2.09"
-      upper="2.09"
-      effort="${motor_torque}"
-      velocity="${motor_vec}" />
-    <dynamics
-      damping="${damping}"
-      friction="${friction}" />
-  </joint>
-  <link
-    name="r_ank_pitch_link">
-    <inertial>
-      <origin
-        xyz="-0.0175439564530261 0.0195631980917168 0.0134182145609028"
-        rpy="0 0 0" />
-      <mass
-        value="0.120" />
-      <inertia
-        ixx="0.00002920"
-        ixy="-0.00000122"
-        ixz="0.00000047"
-        iyy="0.00007365"
-        iyz="0.00000002"
-        izz="0.00006107" />
-    </inertial>
-    <visual>
-      <origin
-        xyz="0 0 0"
-        rpy="0 0 0" />
-      <geometry>
-        <mesh
-          filename="package://ainex_description/meshes/r_ank_pitch_link.STL" />
-      </geometry>
-      <material name="black"/>
-    </visual>
-    <collision>
-      <origin
-        xyz="0 0 0"
-        rpy="0 0 0" />
-      <geometry>
-        <mesh
-          filename="package://ainex_description/meshes/r_ank_pitch_link.STL" />
-      </geometry>
-    </collision>
-  </link>
-  <joint
-    name="r_ank_pitch"
-    type="revolute">
-    <origin
-      xyz="0.0010369887037887 0 -0.0890765640232094"
-      rpy="0 0 0" />
-    <parent
-      link="r_knee_link" />
-    <child
-      link="r_ank_pitch_link" />
-    <axis
-      xyz="0 1 0" />
-    <limit
-      lower="-2.09"
-      upper="2.09"
-      effort="${motor_torque}"
-      velocity="${motor_vec}" />
-    <dynamics
-      damping="${damping}"
-      friction="${friction}" />
-  </joint>
-  <link
-    name="r_ank_roll_link">
-    <inertial>
-      <origin
-        xyz="0.0285084749683582 -0.0128728703698743 -0.0176710108439943"
-        rpy="0 0 0" />
-      <mass
-        value="0.0675" />
-      <inertia
-        ixx="0.00004217"
-        ixy="-0.00000108"
-        ixz="-0.00000226"
-        iyy="0.00009246"
-        iyz="0.00000304"
-        izz="0.00012567" />
-    </inertial>
-    <visual>
-      <origin
-        xyz="0 0 0"
-        rpy="0 0 0" />
-      <geometry>
-        <mesh
-          filename="package://ainex_description/meshes/r_ank_roll_link.STL" />
-      </geometry>
-      <material name="black"/>
-    </visual>
-    <collision>
-      <origin
-        xyz="0 0 0"
-        rpy="0 0 0" />
-      <geometry>
-        <mesh
-          filename="package://ainex_description/meshes/r_ank_roll_link.STL" />
-      </geometry>
-    </collision>
-  </link>
-  <joint
-    name="r_ank_roll"
-    type="revolute">
-    <origin
-      xyz="-0.0190366011761311 0.0199999999998644 0"
-      rpy="0 0 0" />
-    <parent
-      link="r_ank_pitch_link" />
-    <child
-      link="r_ank_roll_link" />
-    <axis
-      xyz="1 0 0" />
-    <limit
-      lower="-2.09"
-      upper="2.09"
-      effort="${motor_torque}"
-      velocity="${motor_vec}" />
-    <dynamics
-      damping="${damping}"
-      friction="${friction}" />
-  </joint>
-  <link
-    name="l_hip_yaw_link">
-    <inertial>
-      <origin
-        xyz="-3.11405684236766E-05 -0.00125722452663508 -0.00137130106826952"
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
File: ainex_project/install/ainex_description/share/ainex_description/robots/ainex.xacro (robot description, xacro)
@@ -1,5 +1 @@
-<?xml version="1.0" encoding="utf-8"?>
-<robot name="ainex" xmlns:xacro="http://ros.org/wiki/xacro">
-    <xacro:include filename="$(find ainex_description)/urdf/ainex.urdf.xacro"/>
-    <xacro:include filename="$(find ainex_description)/urdf/gazebo.xacro" />
-</robot>
+/workspaces/workspaces/Christiano_Roboto/ainex_project/src/ainex_description/robots/ainex.xacro

File: ainex_project/install/ainex_description/share/ainex_description/robots/gazebo.xacro (robot description, xacro)
@@ -1,230 +1 @@
-<?xml version="1.0"?>
-<robot xmlns:xacro="http://ros.org/wiki/xacro">
-  <xacro:property name="M_PI"   value="3.1415926535897931"/>
-  <gazebo>
-    <plugin name="gazebo_ros_control" filename="libgazebo_ros_control.so">
-      <robotNamespace>/</robotNamespace>
-    </plugin>
-    <plugin name="imu_plugin" filename="libgazebo_ros_imu.so">
-      <alwaysOn>true</alwaysOn>
-      <bodyName>imu_link</bodyName>
-      <frameName>imu_link</frameName>
-      <topicName>imu_data</topicName>
-      <serviceName>imu_service</serviceName>
-      <gaussianNoise>0.0</gaussianNoise>
-      <updateRate>0</updateRate>
-      <imu>
-        <noise>
-          <type>gaussian</type>
-          <rate>
-            <mean>0.0</mean>
-            <stddev>2e-4</stddev>
-            <bias_mean>0.0000075</bias_mean>
-            <bias_stddev>0.0000008</bias_stddev>
-          </rate>
-          <accel>
-            <mean>0.0</mean>
-            <stddev>1.7e-2</stddev>
-            <bias_mean>0.1</bias_mean>
-            <bias_stddev>0.001</bias_stddev>
-          </accel>
-        </noise>
-      </imu>
-    </plugin>
-  </gazebo>
-  <gazebo reference="camera_link">
-      <sensor type="camera" name="camera">
-          <update_rate>30.0</update_rate>
-          <camera name="head">
-              <pose>0 0 0 ${M_PI} -${M_PI/2} -${M_PI/2}</pose>
-              <horizontal_fov>1.085595</horizontal_fov>
-              <image>
-                  <width>640</width>
-                  <height>480</height>
-                  <format>R8G8B8</format>
-              </image>
-              <clip>
-                  <near>0.03</near>
-                  <far>100</far>
-              </clip>
-              <noise>
-                  <type>gaussian</type>
-                  <mean>0.0</mean>
-                  <stddev>0.007</stddev>
-              </noise>
-          </camera>
-          <plugin name="gazebo_camera" filename="libgazebo_ros_camera.so">
-              <alwaysOn>true</alwaysOn>
-              <updateRate>0.0</updateRate>
-              <cameraName>/camera</cameraName>
-              <imageTopicName>image_raw</imageTopicName>
-              <cameraInfoTopicName>camera_info</cameraInfoTopicName>
-              <frameName>camera_link</frameName>
-              <hackBaseline>0.07</hackBaseline>
-              <distortionK1>0.0</distortionK1>
-              <distortionK2>0.0</distortionK2>
-              <distortionK3>0.0</distortionK3>
-              <distortionT1>0.0</distortionT1>
-              <distortionT2>0.0</distortionT2>
-          </plugin>
-      </sensor>
-  </gazebo>
-  <gazebo reference="body_link">
-    <mu1>0.2</mu1>
-    <mu2>0.2</mu2>
-    <material>Gazebo/Black</material>
-    <selfCollide>false</selfCollide>
-  </gazebo>
-  <gazebo reference="l_hip_yaw_link">
-    <mu1>0.2</mu1>
-    <mu2>0.2</mu2>
-    <material>Gazebo/Black</material>
-    <selfCollide>false</selfCollide>
-  </gazebo>
-  <gazebo reference="l_hip_roll_link">
-    <mu1>0.2</mu1>
-    <mu2>0.2</mu2>
-    <material>Gazebo/Black</material>
-    <selfCollide>false</selfCollide>
-  </gazebo>
-  <gazebo reference="l_hip_pitch_link">
-    <mu1>0.2</mu1>
-    <mu2>0.2</mu2>
-    <material>Gazebo/Black</material>
-    <selfCollide>false</selfCollide>
-  </gazebo>
-  <gazebo reference="l_knee_link">
-    <mu1>0.2</mu1>
-    <mu2>0.2</mu2>
-    <material>Gazebo/Black</material>
-    <selfCollide>false</selfCollide>
-  </gazebo>
-  <gazebo reference="l_ank_pitch_link">
-    <mu1>0.2</mu1>
-    <mu2>0.2</mu2>
-    <material>Gazebo/Black</material>
-    <selfCollide>false</selfCollide>
-  </gazebo>
-  <gazebo reference="l_ank_roll_link">
-    <kp>100000.0</kp>
-    <kd>100.0</kd>
-    <mu1>1.5</mu1>
-    <mu2>1.5</mu2>
-    <fdir1>1 0 0</fdir1>
-    <maxVel>1.0</maxVel>
-    <minDepth>0.001</minDepth>
-    <material>Gazebo/Black</material>
-  </gazebo>
-  <gazebo reference="r_hip_yaw_link">
-    <mu1>0.2</mu1>
-    <mu2>0.2</mu2>
-    <material>Gazebo/Black</material>
-    <selfCollide>false</selfCollide>
-  </gazebo>
-  <gazebo reference="r_hip_roll_link">
-    <mu1>0.2</mu1>
-    <mu2>0.2</mu2>
-    <material>Gazebo/Black</material>
-    <selfCollide>false</selfCollide>
-  </gazebo>
-  <gazebo reference="r_hip_pitch_link">
-    <mu1>0.2</mu1>
-    <mu2>0.2</mu2>
-    <material>Gazebo/Black</material>
-    <selfCollide>false</selfCollide>
-  </gazebo>
-  <gazebo reference="r_knee_link">
-    <mu1>0.2</mu1>
-    <mu2>0.2</mu2>
-    <material>Gazebo/Black</material>
-    <selfCollide>false</selfCollide>
-  </gazebo>
-  <gazebo reference="r_ank_pitch_link">
-    <mu1>0.2</mu1>
-    <mu2>0.2</mu2>
-    <material>Gazebo/Black</material>
-    <selfCollide>false</selfCollide>
-  </gazebo>
-  <gazebo reference="r_ank_roll_link">
-    <kp>100000.0</kp>
-    <kd>100.0</kd>
-    <mu1>1.5</mu1>
-    <mu2>1.5</mu2>
-    <fdir1>1 0 0</fdir1>
-    <maxVel>1.0</maxVel>
-    <minDepth>0.001</minDepth>
-    <material>Gazebo/Black</material>
-  </gazebo>
-  <gazebo reference="r_sho_pitch_link">
-    <mu1>0.2</mu1>
-    <mu2>0.2</mu2>
-    <material>Gazebo/Black</material>
-    <selfCollide>false</selfCollide>
-  </gazebo>
-  <gazebo reference="r_sho_roll_link">
-    <mu1>0.2</mu1>
-    <mu2>0.2</mu2>
-    <material>Gazebo/Black</material>
-    <selfCollide>false</selfCollide>
-  </gazebo>
-  <gazebo reference="r_el_pitch_link">
-    <mu1>0.2</mu1>
-    <mu2>0.2</mu2>
-    <material>Gazebo/Black</material>
-    <selfCollide>false</selfCollide>
-  </gazebo>
-  <gazebo reference="r_el_yaw_link">
-    <mu1>0.2</mu1>
-    <mu2>0.2</mu2>
-    <material>Gazebo/Black</material>
-    <selfCollide>false</selfCollide>
-  </gazebo>
-  <gazebo reference="r_gripper_link">
-    <mu1>0.2</mu1>
-    <mu2>0.2</mu2>
-    <material>Gazebo/Black</material>
-    <selfCollide>false</selfCollide>
-  </gazebo>
-  <gazebo reference="l_sho_pitch_link">
-    <mu1>0.2</mu1>
-    <mu2>0.2</mu2>
-    <material>Gazebo/Black</material>
-    <selfCollide>false</selfCollide>
-  </gazebo>
-  <gazebo reference="l_sho_roll_link">
-    <mu1>0.2</mu1>
-    <mu2>0.2</mu2>
-    <material>Gazebo/Black</material>
-    <selfCollide>false</selfCollide>
-  </gazebo>
-  <gazebo reference="l_el_pitch_link">
-    <mu1>0.2</mu1>
-    <mu2>0.2</mu2>
-    <material>Gazebo/Black</material>
-    <selfCollide>false</selfCollide>
-  </gazebo>
-  <gazebo reference="l_el_yaw_link">
-    <mu1>0.2</mu1>
-    <mu2>0.2</mu2>
-    <material>Gazebo/Black</material>
-    <selfCollide>false</selfCollide>
-  </gazebo>
-  <gazebo reference="l_gripper_link">
-    <mu1>0.2</mu1>
-    <mu2>0.2</mu2>
-    <material>Gazebo/Black</material>
-    <selfCollide>false</selfCollide>
-  </gazebo>
-  <gazebo reference="head_pan_link">
-    <mu1>0.2</mu1>
-    <mu2>0.2</mu2>
-    <material>Gazebo/Black</material>
-    <selfCollide>false</selfCollide>
-  </gazebo>
-  <gazebo reference="head_tilt_link">
-    <mu1>0.2</mu1>
-    <mu2>0.2</mu2>
-    <material>Gazebo/Black</material>
-    <selfCollide>false</selfCollide>
-  </gazebo>
-</robot>
+/workspaces/workspaces/Christiano_Roboto/ainex_project/src/ainex_description/robots/gazebo.xacro

File: ainex_project/install/ainex_description/share/ainex_description/robots/materials.xacro (robot description, xacro)
@@ -1,27 +1 @@
-<?xml version="1.0"?>
-<robot>
-    <material name="black">
-        <color rgba="0.1 0.1 0.1 1.0"/>
-    </material>
-    <material name="blue">
-        <color rgba="0.0 0.0 0.8 1.0"/>
-    </material>
-    <material name="green">
-        <color rgba="0.4 0.9 0.4 1.0"/>
-    </material>
-    <material name="gray">
-        <color rgba="0.7 0.7 0.7 1.0"/>
-    </material>
-    <material name="darkgray">
-        <color rgba="0.3 0.3 0.3 1.0"/>
-    </material>
-    <material name="red">
-        <color rgba="0.8 0.0 0.0 1.0"/>
-    </material>
-    <material name="white">
-        <color rgba="1.0 1.0 1.0 1.0"/>
-    </material>
-    <material name="yellow">
-        <color rgba="0.8 0.8 0.0 1.0"/>
-    </material>
-</robot>
+/workspaces/workspaces/Christiano_Roboto/ainex_project/src/ainex_description/robots/materials.xacro

File: ainex_project/install/ainex_description/share/ainex_description/robots/transmissions.xacro (robot description, xacro)
@@ -1,42 +1 @@
-<?xml version="1.0"?>
-<robot xmlns:xacro="http://ros.org/wiki/xacro">
-  <xacro:macro name="insert_transmission" params="name">
-    <transmission name="${name}_tran">
-      <type>transmission_interface/SimpleTransmission</type>
-      <joint name="${name}">
-        <hardwareInterface>hardware_interface/EffortJointInterface</hardwareInterface>
-      </joint>
-      <actuator name="${name}_motor">
-        <hardwareInterface>hardware_interface/EffortJointInterface</hardwareInterface>
-        <mechanicalReduction>1</mechanicalReduction>
-      </actuator>
-    </transmission>
-  </xacro:macro>
-  <!--leg-->
-  <xacro:insert_transmission name="l_hip_roll" />
-  <xacro:insert_transmission name="l_hip_pitch" />
-  <xacro:insert_transmission name="r_hip_roll" />
-  <xacro:insert_transmission name="r_hip_pitch" />
-  <xacro:insert_transmission name="l_hip_yaw" />
-  <xacro:insert_transmission name="r_hip_yaw" />
-  <xacro:insert_transmission name="l_knee" />
-  <xacro:insert_transmission name="l_ank_pitch" />
-  <xacro:insert_transmission name="l_ank_roll" />
-  <xacro:insert_transmission name="r_knee" />
-  <xacro:insert_transmission name="r_ank_pitch" />
-  <xacro:insert_transmission name="r_ank_roll" />
-  <!--arm-->
-  <xacro:insert_transmission name="l_sho_roll" />
-  <xacro:insert_transmission name="l_sho_pitch" />
-  <xacro:insert_transmission name="r_sho_roll" />
-  <xacro:insert_transmission name="r_sho_pitch" />
-  <xacro:insert_transmission name="l_el_yaw" />
-  <xacro:insert_transmission name="r_el_yaw" />
-  <xacro:insert_transmission name="l_el_pitch" />
-  <xacro:insert_transmission name="l_gripper" />
-  <xacro:insert_transmission name="r_el_pitch" />
-  <xacro:insert_transmission name="r_gripper" />
-  <!--head-->
-  <xacro:insert_transmission name="head_pan" />
-  <xacro:insert_transmission name="head_tilt" />
-</robot>
+/workspaces/workspaces/Christiano_Roboto/ainex_project/src/ainex_description/robots/transmissions.xacro
