Commit message: Theresa: changed urdf to zero position of hardware robot

File: ainex_project/src/ainex_description/robots/ainex.urdf (robot description, URDF)
Before this commit: robot ainex, 28 links, 27 joints
Joints:
- joint l_sho_roll: origin xyz=0.020003 0.021507 0 rpy=0 0 0 -> xyz=0.020003 0.021507 0 rpy=-1.5708 0 0
- joint r_sho_roll: origin xyz=0.020003499818653 -0.021505961295104 0 rpy=0 0 0 -> xyz=0.020003499818653 -0.021505961295104 0 rpy=1.5708 0 0
